File: converter.sch (KiCad schematic (older format))
At the start: 30 parts, among them J1 USB_B, K1 PS2_FEMALE, K2 ADB_FEMALE, K3 CONN_3, P1 CONN_5, P10 CONN_4, P2 CONN_8, P3 CONN_8, P4 CONN_1, P5 CONN_1, P6 CONN_1, P7 CONN_1, P8 CONN_1, P9 CONN_1, SW1 SW_PUSH, U1 ATMEGA32U4, X1 16MHz

Commit message: Add converter.mod
Parts:
- removed K1: PS2_FEMALE, symbol PS2_FEMALE
- removed K2: ADB_FEMALE, symbol ADB_FEMALE
- removed K3: CONN_3, symbol CONN_3
- removed P1: CONN_5, symbol CONN_5
- removed P10: CONN_4, symbol CONN_4
- removed P2, P3: CONN_8, symbol CONN_8
- added CN1: MINI_DIN_8P_JACK, symbol MINI_DIN_8P_JACK
- added P1, P10, P11, P12, P13, P14, P15, P16, P17, P18, P19, P2, P20, P21, P22, P23, P24, P25, P26, P27, P28, P29, P3, P30, P31, P32, P33, P34, P35, P36, P4, P5, P6, P7, P8, P9: CONN_1, symbol CONN_1
- added R5, R6, R7, R8: 1K, symbol R
- renumbered P4 to P37, P5 to P38, P6 to P39, P7 to P40, P8 to P41, P9 to P42
Connections:
- net labels added: DIN1, DIN2, DIN3, DIN4, DIN5, DIN6, DIN7, DIN8
- wire segments 115 -> 132
Other:
- note added: "Controller I/O Pins"
- note added: "Mini DIN connector(4-8P)\n4: ADB\n6: PS/2\n7: X68000\n8: SUN, PC98"
- note added: "Pullup Resistors"
- note added: "USB pins for external connector"
- moved on the sheet: P37, P38, P39, P40, P41, P42

Commit message: Wire component
Other:
- note added: "+/-5%"
- note added: "Ucap +/-10%"
Changed lines of the file:
@@
-EESchema Schematic File Version 2  date 2013年04月30日 16時39分43秒
+EESchema Schematic File Version 2  date 2013年05月02日 10時58分37秒
 LIBS:power
 LIBS:device
@@
 Sheet 1 1
 Title "Keyboard Converter"
-Date "30 apr 2013"
+Date "2 may 2013"
 Rev "1.0"
 Comp ""
@@
 $EndComp
 $Comp
-L PWR_FLAG #FLG1
+L PWR_FLAG #FLG01
 U 1 1 4EBBEFCE
 P 750 7600
-F 0 "#FLG1" H 750 7870 30  0001 C CNN
+F 0 "#FLG01" H 750 7870 30  0001 C CNN
 F 1 "PWR_FLAG" H 750 7830 30  0000 C CNN
 F 2 "" H 750 7600 60  0001 C CNN
@@
 $EndComp
 $Comp
-L GND #PWR1
+L GND #PWR02
 U 1 1 4EBBEF66
 P 750 7600
-F 0 "#PWR1" H 750 7600 30  0001 C CNN
+F 0 "#PWR02" H 750 7600 30  0001 C CNN
 F 1 "GND" H 750 7530 30  0001 C CNN
 F 2 "" H 750 7600 60  0001 C CNN
@@
 $EndComp
 $Comp
-L GND #PWR7
+L GND #PWR03
 U 1 1 4EBA913C
 P 5300 4400
-F 0 "#PWR7" H 5300 4400 30  0001 C CNN
+F 0 "#PWR03" H 5300 4400 30  0001 C CNN
 F 1 "GND" H 5300 4330 30  0001 C CNN
 F 2 "" H 5300 4400 60  0001 C CNN
@@
 $EndComp
 $Comp
-L GND #PWR13
+L GND #PWR04
 U 1 1 4EBA912C
 P 6600 4400
-F 0 "#PWR13" H 6600 4400 30  0001 C CNN
+F 0 "#PWR04" H 6600 4400 30  0001 C CNN
 F 1 "GND" H 6600 4330 30  0001 C CNN
 F 2 "" H 6600 4400 60  0001 C CNN
@@
 $EndComp
 $Comp
-L GND #PWR17
+L GND #PWR05
 U 1 1 4EBA35B3
 P 9800 4400
-F 0 "#PWR17" H 9800 4400 30  0001 C CNN
+F 0 "#PWR05" H 9800 4400 30  0001 C CNN
 F 1 "GND" H 9800 4330 30  0001 C CNN
 F 2 "" H 9800 4400 60  0001 C CNN
@@
 $EndComp
 $Comp
-L GND #PWR19
+L GND #PWR06
 U 1 1 4EBA3599
 P 10300 4400
-F 0 "#PWR19" H 10300 4400 30  0001 C CNN
+F 0 "#PWR06" H 10300 4400 30  0001 C CNN
 F 1 "GND" H 10300 4330 30  0001 C CNN
 F 2 "" H 10300 4400 60  0001 C CNN
@@
 $EndComp
 $Comp
-L GND #PWR3
+L GND #PWR07
 U 1 1 4EBA3538
 P 3200 2950
-F 0 "#PWR3" H 3200 2950 30  0001 C CNN
+F 0 "#PWR07" H 3200 2950 30  0001 C CNN
 F 1 "GND" H 3200 2880 30  0001 C CNN
 F 2 "" H 3200 2950 60  0001 C CNN
@@
 $EndComp
 $Comp
-L GND #PWR18
+L GND #PWR08
 U 1 1 4EBA3506
 P 10050 4400
-F 0 "#PWR18" H 10050 4400 30  0001 C CNN
+F 0 "#PWR08" H 10050 4400 30  0001 C CNN
 F 1 "GND" H 10050 4330 30  0001 C CNN
 F 2 "" H 10050 4400 60  0001 C CNN
@@
 $EndComp
 $Comp
-L GND #PWR16
+L GND #PWR09
 U 1 1 4EBA3501
 P 9550 4400
-F 0 "#PWR16" H 9550 4400 30  0001 C CNN
+F 0 "#PWR09" H 9550 4400 30  0001 C CNN
 F 1 "GND" H 9550 4330 30  0001 C CNN
 F 2 "" H 9550 4400 60  0001 C CNN
@@
 $EndComp
 $Comp
-L GND #PWR14
+L GND #PWR010
 U 1 1 4EBA34E8
 P 9250 4400
-F 0 "#PWR14" H 9250 4400 30  0001 C CNN
+F 0 "#PWR010" H 9250 4400 30  0001 C CNN
 F 1 "GND" H 9250 4330 30  0001 C CNN
 F 2 "" H 9250 4400 60  0001 C CNN
@@
 $EndComp
 $Comp
-L GND #PWR11
+L GND #PWR011
 U 1 1 4EBA3454
 P 6300 4400
-F 0 "#PWR11" H 6300 4400 30  0001 C CNN
+F 0 "#PWR011" H 6300 4400 30  0001 C CNN
 F 1 "GND" H 6300 4330 30  0001 C CNN
 F 2 "" H 6300 4400 60  0001 C CNN
@@
 $EndComp
 $Comp
-L +5V #PWR15
+L +5V #PWR012
 U 1 1 4EBA2BA0
 P 9550 1550
-F 0 "#PWR15" H 9550 1520 20  0001 C CNN
+F 0 "#PWR012" H 9550 1520 20  0001 C CNN
 F 1 "+5V" H 9550 1660 30  0000 C CNN
 F 2 "" H 9550 1550 60  0001 C CNN
@@
 $EndComp
 $Comp
-L +5V #PWR5
+L +5V #PWR013
 U 1 1 4EBA2B28
 P 5050 1550
-F 0 "#PWR5" H 5050 1520 20  0001 C CNN
+F 0 "#PWR013" H 5050 1520 20  0001 C CNN
 F 1 "+5V" H 5050 1660 30  0000 C CNN
 F 2 "" H 5050 1550 60  0001 C CNN
@@
 $EndComp
 $Comp
-L +5V #PWR12
+L +5V #PWR014
 U 1 1 4EBA2B15
 P 6600 1550
-F 0 "#PWR12" H 6600 1520 20  0001 C CNN
+F 0 "#PWR014" H 6600 1520 20  0001 C CNN
 F 1 "+5V" H 6600 1660 30  0000 C CNN
 F 2 "" H 6600 1550 60  0001 C CNN
@@
 VCC
 $Comp
-L +5V #PWR2
+L +5V #PWR015
 U 1 1 4EB8CC7B
 P 3200 1550
-F 0 "#PWR2" H 3200 1520 20  0001 C CNN
+F 0 "#PWR015" H 3200 1520 20  0001 C CNN
 F 1 "+5V" H 3200 1660 30  0000 C CNN
 F 2 "" H 3200 1550 60  0001 C CNN
@@
 $EndComp
 $Comp
-L GND #PWR6
+L GND #PWR016
 U 1 1 4EB8BB5A
 P 5050 4400
-F 0 "#PWR6" H 5050 4400 30  0001 C CNN
+F 0 "#PWR016" H 5050 4400 30  0001 C CNN
 F 1 "GND" H 5050 4330 30  0001 C CNN
 F 2 "" H 5050 4400 60  0001 C CNN
@@
 ~RESET
 $Comp
-L GND #PWR8
+L GND #PWR017
 U 1 1 4EB8BB49
 P 5500 2950
-F 0 "#PWR8" H 5500 2950 30  0001 C CNN
+F 0 "#PWR017" H 5500 2950 30  0001 C CNN
 F 1 "GND" H 5500 2880 30  0001 C CNN
 F 2 "" H 5500 2950 60  0001 C CNN
@@
 $EndComp
 $Comp
-L GND #PWR9
+L GND #PWR018
 U 1 1 4EB8BB48
 P 5500 4400
-F 0 "#PWR9" H 5500 4400 30  0001 C CNN
+F 0 "#PWR018" H 5500 4400 30  0001 C CNN
 F 1 "GND" H 5500 4330 30  0001 C CNN
 F 2 "" H 5500 4400 60  0001 C CNN
@@
 $EndComp
 $Comp
-L GND #PWR10
+L GND #PWR019
 U 1 1 4EB8BB47
 P 5700 4400
-F 0 "#PWR10" H 5700 4400 30  0001 C CNN
+F 0 "#PWR019" H 5700 4400 30  0001 C CNN
 F 1 "GND" H 5700 4330 30  0001 C CNN
 F 2 "" H 5700 4400 60  0001 C CNN
@@
 $EndComp
 $Comp
-L +5V #PWR4
+L +5V #PWR020
 U 1 1 517F6E08
 P 5400 4800
-F 0 "#PWR4" H 5400 4890 20  0001 C CNN
+F 0 "#PWR020" H 5400 4890 20  0001 C CNN
 F 1 "+5V" H 5400 4890 30  0000 C CNN
 F 2 "" H 5400 4800 60  0000 C CNN
@@
 Text Notes 8200 5850 0    60   Italic 0
 Controller I/O Pins
+Text Notes 5700 2750 0    60   Italic 0
+Ucap +/-10%
+Text Notes 3850 2450 0    60   Italic 0
++/-5%
 $EndSCHEMATC

Commit message: Rev1 for fusion PCB
Parts:
- removed C6: 0.1u, symbol C
- removed R3: 10K, symbol R
- added D1: LED, symbol LED
- added R8: 1K, symbol R
- renumbered C7 to C6, C8 to C7, C9 to C8, R4 to R3, R5 to R4, R6 to R5, R7 to R6, R8 to R7
Connections:
- wire segments 132 -> 133
Other:
- note added: "Optional Teensy compatible LED"
- moved on the sheet: CN1, P10, P11, P12, P5, P6, P7, P8, P9, R4, R5, R6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
