File: converter.sch (KiCad schematic (older format))
At the start: 64 parts, among them CN1 MINI_DIN_8P_JACK, J1 USB_B, P1 CONN_1, P10 CONN_1, P11 CONN_1, P12 CONN_1, P13 CONN_1, P14 CONN_1, P15 CONN_1, P16 CONN_1, P17 CONN_1, P18 CONN_1, P19 CONN_1, P2 CONN_1, P20 CONN_1, P21 CONN_1, P22 CONN_1, P23 CONN_1, P24 CONN_1, P25 CONN_1, P26 CONN_1, P27 CONN_1, P28 CONN_1, P29 CONN_1, P3 CONN_1, P30 CONN_1, P31 CONN_1, P32 CONN_1, P33 CONN_1, P34 CONN_1, P35 CONN_1, P36 CONN_1, P37 CONN_1, P38 CONN_1, P39 CONN_1, P4 CONN_1, P40 CONN_1, P41 CONN_1, P42 CONN_1, P5 CONN_1, P6 CONN_1, P7 CONN_1, P8 CONN_1, P9 CONN_1, SW1 SW_PUSH, U1 ATMEGA32U4, X1 16MHz

Commit message: Initial commit of PCB rev.2
Parts:
- removed C6, C7, C8: 0.1u, symbol C
- removed J1: USB_B, symbol USB_MINIB
- removed P10, P11, P12, P13, P14, P15, P16, P17, P18, P19, P20, P21, P22, P23, P24, P25, P26, P27, P28, P29, P30, P31, P32, P33, P34, P35, P36, P37, P38, P39, P40, P41, P42, P5, P6, P7, P8, P9: CONN_1, symbol CONN_1
- removed U1: ATMEGA32U4, symbol ATMEGA32U4
- added C4: 0.1u, symbol C
- added J1: USB_mini_micro_B, symbol USB_mini_micro_B
- added R14: 1K, symbol R
- added SJ1, SJ10, SJ11, SJ12, SJ13, SJ14, SJ15, SJ16, SJ17, SJ18, SJ19, SJ2, SJ20, SJ21, SJ22, SJ23, SJ24, SJ25, SJ26, SJ27, SJ28, SJ29, SJ3, SJ30, SJ4, SJ5, SJ6, SJ7, SJ8, SJ9, SJ98, SJ99: SOLDER_JUMPER, symbol SOLDER_JUMPER
- added U1: ATMEGA32U2, symbol ATMEGA32U2
- renumbered C4 to C5, C5 to C6, R4 to R10, R5 to R11, R6 to R12, R7 to R13, R8 to R4
Connections:
- net labels added: PC2, PC4, PC5
- net labels removed: AREF, PE6, PF0, PF1, PF4, PF5, PF6, PF7
- wire segments 133 -> 184
- no-connect marks 0 -> 15
Other:
- note added: "+-5%"
- note added: "ADB"
- note added: "Keyboard Connector"
- note added: "Mini DIN connector\n4P: ADB\n5P: NEXT\n6P: PS/2\n7P: X68000\n8P: SUN, PC98"
- note added: "NEXT"
- note added: "Optional\nTeensy compatible LED"
- note added: "PC98"
- note added: "PS/2"
- note added: "Pin Configuration"
- note added: "Pinout"
- note added: "SUN"
- note added: "USB"
- note added: "X68K"
- note removed: "+/-5%"
- note removed: "Controller I/O Pins"
- note removed: "Mini DIN connector(4-8P)\n4: ADB\n6: PS/2\n7: X68000\n8: SUN, PC98"
- note removed: "Optional Teensy compatible LED"
- note removed: "USB pins for external connector"
- moved on the sheet: C1, C2, C3, C5, C6, D1, P1, P2, P3, P4, R1, R10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

Commit message: rev2.1
Changed lines of the file:
@@
 LIBS:keyboard_parts
 LIBS:converter-cache
-LIBS:power
-LIBS:device
-LIBS:transistors
-LIBS:conn
-LIBS:linear
-LIBS:regul
-LIBS:74xx
-LIBS:cmos4000
-LIBS:adc-dac
-LIBS:memory
-LIBS:xilinx
-LIBS:special
-LIBS:microcontrollers
-LIBS:dsp
-LIBS:microchip
-LIBS:analog_switches
-LIBS:motorola
-LIBS:texas
-LIBS:intel
-LIBS:audio
-LIBS:interface
-LIBS:digital-audio
-LIBS:philips
-LIBS:display
-LIBS:cypress
-LIBS:siliconi
-LIBS:opto
-LIBS:atmel
-LIBS:contrib
-LIBS:valves
-LIBS:atmega32u2
-LIBS:solder_jumper
-LIBS:mini_din_8p_jack
 LIBS:converter-cache
 EELAYER 24 0
@@
 	1    0    0    -1
 $EndComp
+NoConn ~ 2100 2175
+NoConn ~ 2100 2575
+NoConn ~ 2100 2675
+NoConn ~ 4250 2675
+$Comp
+L CRYSTAL X1
+U 1 1 532E55A0
+P 1050 1625
+F 0 "X1" H 1050 1775 60  0000 C CNN
+F 1 "16MHz" H 1050 1475 60  0000 C CNN
+F 2 "" H 1050 1625 60  0000 C CNN
+F 3 "" H 1050 1625 60  0000 C CNN
+	1    1050 1625
+	1    0    0    -1
+$EndComp
 Wire Wire Line
 	2100 2675 1850 2675
@@
 Connection ~ 5750 1675
 Connection ~ 6150 1675
-Connection ~ 6150 1775
 Wire Wire Line
 	725  7325 725  7375
@@
 Wire Notes Line
 	4200 6600 4200 7750
-NoConn ~ 2100 2175
-NoConn ~ 2100 2575
-NoConn ~ 2100 2675
-NoConn ~ 4250 2675
+Wire Wire Line
+	725  7625 725  7675
+Wire Notes Line
+	3150 6325 3150 7750
+Wire Notes Line
+	3225 6600 4200 6600
+Wire Wire Line
+	5900 1775 5750 1775
+Connection ~ 5750 1775
+Wire Wire Line
+	1050 1825 1050 1925
 $Comp
 L SOLDER_JUMPER SJ99
-U 1 1 532E48D4
+U 1 1 53A52D85
 P 675 7475
 F 0 "SJ99" H 675 7425 60  0000 C CNN
@@
 	0    1    1    0
 $EndComp
-Wire Wire Line
-	725  7625 725  7675
-Wire Notes Line
-	3150 6325 3150 7750
-Wire Notes Line
-	3225 6600 4200 6600
 $Comp
 L SOLDER_JUMPER SJ98
-U 1 1 532E530F
+U 1 1 53A52524
 P 6000 1825
 F 0 "SJ98" H 6000 1775 60  0000 C CNN
@@
 	1    0    0    -1
 $EndComp
-Wire Wire Line
-	5900 1775 5750 1775
-Connection ~ 5750 1775
-$Comp
-L CRYSTAL X1
-U 1 1 532E55A0
-P 1050 1625
-F 0 "X1" H 1050 1775 60  0000 C CNN
-F 1 "16MHz" H 1050 1475 60  0000 C CNN
-F 2 "" H 1050 1625 60  0000 C CNN
-F 3 "" H 1050 1625 60  0000 C CNN
-	1    1050 1625
-	1    0    0    -1
-$EndComp
-Wire Wire Line
-	1050 1825 1050 1925
 $EndSCHEMATC

Commit message: Change values of capacitors and solder mask setting
Parts:
- C1: value 10u -> 4.7u
- C5, C6: value 22p -> 10p
Changed lines of the file:
@@
 LIBS:keyboard_parts
 LIBS:converter-cache
-LIBS:converter-cache
-EELAYER 24 0
+EELAYER 25 0
 EELAYER END
 $Descr A4 11693 8268
@@
 Sheet 1 1
 Title "TMK Keyboard Converter - Mini DIN"
-Date "2014/03"
-Rev "2.0"
+Date "2015/12"
+Rev "2.3"
 Comp "hasu@TMK"
 Comment1 ""
@@
 P 6125 2425
 F 0 "C1" H 6175 2525 50  0000 L CNN
-F 1 "10u" H 6175 2325 50  0000 L CNN
+F 1 "4.7u" H 6175 2325 50  0000 L CNN
 F 2 "" H 6125 2425 60  0001 C CNN
 F 3 "" H 6125 2425 60  0001 C CNN
@@
 P 750 1875
 F 0 "C5" H 800 1975 50  0000 L CNN
-F 1 "22p" H 800 1775 50  0000 L CNN
+F 1 "10p" H 800 1775 50  0000 L CNN
 F 2 "" H 750 1875 60  0001 C CNN
 F 3 "" H 750 1875 60  0001 C CNN
@@
 P 1350 1875
 F 0 "C6" H 1400 1975 50  0000 L CNN
-F 1 "22p" H 1400 1775 50  0000 L CNN
+F 1 "10p" H 1400 1775 50  0000 L CNN
 F 2 "" H 1350 1875 60  0001 C CNN
 F 3 "" H 1350 1875 60  0001 C CNN
